Commit message: moved  mars_sim and mars_description folders to ros_ws and solved dependecies for ur5 urdf

File: ros_ws/src/mars_description/urdf/mars_robot.urdf.xacro (robot description, xacro)
@@ -130,5 +130,5 @@
   </joint>
   <!-- ur5 -->
-  <xacro:include filename="$(find ur_description)/urdf/ur5.urdf.xacro"/>
+  <xacro:include filename="$(find mars_description)/urdf/ur5.urdf.xacro"/>
   <!-- arm -->
   <xacro:ur5_robot prefix="ur5_" joint_limited="true"/>

File: ros_ws/src/mars_description/urdf/ur5.urdf.xacro (robot description, xacro)
@@ -1,6 +1,6 @@
 <?xml version="1.0"?>
 <robot xmlns:xacro="http://ros.org/wiki/xacro">
-  <xacro:include filename="$(find ur_description)/urdf/ur.transmission.xacro" />
-  <xacro:include filename="$(find ur_description)/urdf/ur.gazebo.xacro" />
+  <xacro:include filename="$(find mars_description)/urdf/ur.transmission.xacro" />
+  <xacro:include filename="$(find mars_description)/urdf/ur.gazebo.xacro" />
   <xacro:property name="pi" value="3.14159265" />
   <!-- Inertia parameters -->
@@ -72,13 +72,13 @@
       <visual>
         <geometry>
-          <mesh filename="package://ur_description/meshes/ur5/visual/base.dae" />
-        </geometry>
-        <material name="LightGrey">
-          <color rgba="0.7 0.7 0.7 1.0"/>
-        </material>
-      </visual>
-      <collision>
-        <geometry>
-          <mesh filename="package://ur_description/meshes/ur5/collision/base.stl" />
+          <mesh filename="package://mars_description/meshes/ur5/visual/base.dae" />
+        </geometry>
+        <material name="LightGrey">
+          <color rgba="0.7 0.7 0.7 1.0"/>
+        </material>
+      </visual>
+      <collision>
+        <geometry>
+          <mesh filename="package://mars_description/meshes/ur5/collision/base.stl" />
         </geometry>
       </collision>
@@ -103,13 +103,13 @@
       <visual>
         <geometry>
-          <mesh filename="package://ur_description/meshes/ur5/visual/shoulder.dae" />
-        </geometry>
-        <material name="LightGrey">
-          <color rgba="0.7 0.7 0.7 1.0"/>
-        </material>
-      </visual>
-      <collision>
-        <geometry>
-          <mesh filename="package://ur_description/meshes/ur5/collision/shoulder.stl" />
+          <mesh filename="package://mars_description/meshes/ur5/visual/shoulder.dae" />
+        </geometry>
+        <material name="LightGrey">
+          <color rgba="0.7 0.7 0.7 1.0"/>
+        </material>
+      </visual>
+      <collision>
+        <geometry>
+          <mesh filename="package://mars_description/meshes/ur5/collision/shoulder.stl" />
         </geometry>
       </collision>
@@ -134,13 +134,13 @@
       <visual>
         <geometry>
-          <mesh filename="package://ur_description/meshes/ur5/visual/upperarm.dae" />
-        </geometry>
-        <material name="LightGrey">
-          <color rgba="0.7 0.7 0.7 1.0"/>
-        </material>
-      </visual>
-      <collision>
-        <geometry>
-          <mesh filename="package://ur_description/meshes/ur5/collision/upperarm.stl" />
+          <mesh filename="package://mars_description/meshes/ur5/visual/upperarm.dae" />
+        </geometry>
+        <material name="LightGrey">
+          <color rgba="0.7 0.7 0.7 1.0"/>
+        </material>
+      </visual>
+      <collision>
+        <geometry>
+          <mesh filename="package://mars_description/meshes/ur5/collision/upperarm.stl" />
         </geometry>
       </collision>
@@ -165,13 +165,13 @@
       <visual>
         <geometry>
-          <mesh filename="package://ur_description/meshes/ur5/visual/forearm.dae" />
-        </geometry>
-        <material name="LightGrey">
-          <color rgba="0.7 0.7 0.7 1.0"/>
-        </material>
-      </visual>
-      <collision>
-        <geometry>
-          <mesh filename="package://ur_description/meshes/ur5/collision/forearm.stl" />
+          <mesh filename="package://mars_description/meshes/ur5/visual/forearm.dae" />
+        </geometry>
+        <material name="LightGrey">
+          <color rgba="0.7 0.7 0.7 1.0"/>
+        </material>
+      </visual>
+      <collision>
+        <geometry>
+          <mesh filename="package://mars_description/meshes/ur5/collision/forearm.stl" />
         </geometry>
       </collision>
@@ -196,13 +196,13 @@
       <visual>
         <geometry>
-          <mesh filename="package://ur_description/meshes/ur5/visual/wrist1.dae" />
-        </geometry>
-        <material name="LightGrey">
-          <color rgba="0.7 0.7 0.7 1.0"/>
-        </material>
-      </visual>
-      <collision>
-        <geometry>
-          <mesh filename="package://ur_description/meshes/ur5/collision/wrist1.stl" />
+          <mesh filename="package://mars_description/meshes/ur5/visual/wrist1.dae" />
+        </geometry>
+        <material name="LightGrey">
+          <color rgba="0.7 0.7 0.7 1.0"/>
+        </material>
+      </visual>
+      <collision>
+        <geometry>
+          <mesh filename="package://mars_description/meshes/ur5/collision/wrist1.stl" />
         </geometry>
       </collision>
@@ -227,13 +227,13 @@
       <visual>
         <geometry>
-          <mesh filename="package://ur_description/meshes/ur5/visual/wrist2.dae" />
-        </geometry>
-        <material name="LightGrey">
-          <color rgba="0.7 0.7 0.7 1.0"/>
-        </material>
-      </visual>
-      <collision>
-        <geometry>
-          <mesh filename="package://ur_description/meshes/ur5/collision/wrist2.stl" />
+          <mesh filename="package://mars_description/meshes/ur5/visual/wrist2.dae" />
+        </geometry>
+        <material name="LightGrey">
+          <color rgba="0.7 0.7 0.7 1.0"/>
+        </material>
+      </visual>
+      <collision>
+        <geometry>
+          <mesh filename="package://mars_description/meshes/ur5/collision/wrist2.stl" />
         </geometry>
       </collision>
@@ -258,13 +258,13 @@
       <visual>
         <geometry>
-          <mesh filename="package://ur_description/meshes/ur5/visual/wrist3.dae" />
-        </geometry>
-        <material name="LightGrey">
-          <color rgba="0.7 0.7 0.7 1.0"/>
-        </material>
-      </visual>
-      <collision>
-        <geometry>
-          <mesh filename="package://ur_description/meshes/ur5/collision/wrist3.stl" />
+          <mesh filename="package://mars_description/meshes/ur5/visual/wrist3.dae" />
+        </geometry>
+        <material name="LightGrey">
+          <color rgba="0.7 0.7 0.7 1.0"/>
+        </material>
+      </visual>
+      <collision>
+        <geometry>
+          <mesh filename="package://mars_description/meshes/ur5/collision/wrist3.stl" />
         </geometry>
       </collision>
@@ -276,5 +276,5 @@
       <parent link="${prefix}wrist_3_link" />
       <child link = "${prefix}ee_link" />
-      <origin xyz="0.0 ${wrist_3_length} 0.0" rpy="${pi/-2.0} 0.0 0.0"/>
+      <origin xyz="0.0 ${wrist_3_length} 0.0" rpy="0.0 0.0 ${pi/2.0}" />
     </joint>
     <link name="${prefix}ee_link">
@@ -283,5 +283,5 @@
           <box size="0.01 0.01 0.01"/>
         </geometry>
-        <origin rpy="${pi/-2.0} 0 0" xyz="0.01 0 0"/>
+        <origin rpy="0 0 0" xyz="-0.01 0 0"/>
       </collision>
     </link>
@@ -295,5 +295,6 @@
                  degrees)
       -->
-    <origin xyz="0 0 0" rpy="0 0 ${-pi}"/>
+      <origin xyz="0 0 0" rpy="0 0 ${-pi}"/>
+      <!--origin xyz="0 0 0" rpy="0 0 0"/-->
       <parent link="${prefix}base_link"/>
       <child link="${prefix}base"/>
@@ -302,5 +303,5 @@
     <link name="${prefix}tool0"/>
     <joint name="${prefix}wrist_3_link-tool0_fixed_joint" type="fixed">
-      <origin xyz="0 ${wrist_3_length + 0.17389} 0" rpy="${pi/-2.0} 0 0"/>
+      <origin xyz="0 ${wrist_3_length} 0" rpy="${pi/-2.0} 0 0"/>
       <parent link="${prefix}wrist_3_link"/>
       <child link="${prefix}tool0"/>
